Commit message: fixed bugs and cleaned up urdf export

File: cad/urdf/bassie_urdf/bassie.urdf (robot description, URDF)
Before this commit: robot bassie.SLDASM, 11 links, 10 joints
Links:
- removed link base_link
- removed link left_foot
- removed link right_foot
- added link left_ankle, mass 0.0141163998019808; collision mesh filename=/meshes/left_ankle.STL; visual mesh filename=/meshes/left_ankle.STL
- added link pelvis, mass 0.030372; collision mesh filename=/meshes/pelvis.STL; visual mesh filename=/meshes/pelvis.STL
- added link right_ankle, mass 0.014116; collision mesh filename=/meshes/right_ankle.STL; visual mesh filename=/meshes/right_ankle.STL
- link left_hip_pitch: geometry collision mesh filename=/meshes/left_hip_pitch.STL; visual mesh filename=/meshes/left_hip_pitch.STL
- link left_hip_roll: mass 0.0104219467105846 -> 0.010422; geometry collision mesh filename=/meshes/left_hip_roll.STL; visual mesh filename=/meshes/left_hip_roll.STL
- link left_hip_yaw: mass 0.107025089754586 -> 0.107042315965997; geometry collision mesh filename=/meshes/left_hip_yaw.STL; visual mesh filename=/meshes/left_hip_yaw.STL
- link left_knee: mass 0.0744483691081149 -> 0.0744483650191621; geometry collision mesh filename=/meshes/left_knee.STL; visual mesh filename=/meshes/left_knee.STL
- link right_hip_pitch: mass 0.0104219467105846 -> 0.010422; geometry collision mesh filename=/meshes/right_hip_pitch.STL; visual mesh filename=/meshes/right_hip_pitch.STL
- link right_hip_roll: geometry collision mesh filename=/meshes/right_hip_roll.STL; visual mesh filename=/meshes/right_hip_roll.STL
- link right_hip_yaw: mass 0.107018899099017 -> 0.10702; geometry collision mesh filename=/meshes/right_hip_yaw.STL; visual mesh filename=/meshes/right_hip_yaw.STL
- link right_knee: mass 0.0744483035148738 -> 0.074448; geometry collision mesh filename=/meshes/right_knee.STL; visual mesh filename=/meshes/right_knee.STL
Joints:
- removed joint left_foot
- removed joint right_foot
- added joint left_ankle: type revolute, parent left_knee, child left_ankle, origin xyz=0 -0.18 0 rpy=-0.090229 0 0, axis 1 0 0, limit lower=-2 upper=2 effort=100 velocity=100
- added joint right_ankle: type revolute, parent right_knee, child right_ankle, origin xyz=0 -0.18 0 rpy=-0.17083 0 0, axis 1 0 0, limit lower=-2 upper=2 effort=100 velocity=100
- joint left_hip_pitch: limit (none) -> lower=-1 upper=1 effort=100 velocity=100; origin xyz=0 -0.0148419385448798 -0.022 rpy=-1.57079632679543 1.55465607457052 0 -> xyz=0 -0.014842 -0.022 rpy=-1.5708 1.5547 0; type continuous -> revolute
- joint left_hip_roll: limit (none) -> lower=-1 upper=1 effort=100 velocity=100; origin xyz=0.0398271658880066 0 -0.00930710361371742 rpy=1.5707963267949 0.214726254431021 0 -> xyz=0.039827 0 -0.0093071 rpy=1.5708 0.21473 0; parent base_link -> pelvis; type continuous -> revolute
- joint left_hip_yaw: limit (none) -> lower=-2 upper=2 effort=100 velocity=100; origin xyz=0 0 -0.0291580614551205 rpy=1.4219328867289 0 -1.5707963267949 -> xyz=0 0 -0.029158 rpy=1.4219 0 -1.5708; type continuous -> revolute
- joint left_knee: limit (none) -> lower=-2 upper=2 effort=100 velocity=100; origin xyz=0.0214112408562416 -0.141421356237311 0.141421356237309 rpy=0.161421391587217 0 0 -> xyz=0.021411 -0.14142 0.14142 rpy=0.16142 0 0; type continuous -> revolute
- joint right_hip_pitch: limit (none) -> lower=-1 upper=1 effort=100 velocity=100; origin xyz=0 -0.0220008611326573 -0.0219999999999999 rpy=-1.57079632679503 -1.49330843492653 0 -> xyz=0 -0.022001 -0.022 rpy=-1.5708 -1.4933 0; type continuous -> revolute
- joint right_hip_roll: limit (none) -> lower=-1 upper=1 effort=100 velocity=100; origin xyz=-0.0398271658880066 0 -0.00930710361371741 rpy=1.5707963267949 -0.00503265783860925 0 -> xyz=-0.039827 0 -0.0093071 rpy=1.5708 -0.0050327 0; parent base_link -> pelvis; type continuous -> revolute
- joint right_hip_yaw: limit (none) -> lower=-2 upper=2 effort=100 velocity=100; origin xyz=0 -0.0210679578739459 -0.0219991388673428 rpy=1.47617469063059 0 1.5707963267949 -> xyz=0 -0.021068 -0.021999 rpy=1.4762 0 1.5708; type continuous -> revolute
- joint right_knee: limit (none) -> lower=-2 upper=2 effort=100 velocity=100; origin xyz=0 -0.14142135623731 0.141421356237308 rpy=0.177493987253612 0 0 -> xyz=0 -0.14142 0.14142 rpy=0.17749 0 0; type continuous -> revolute

Commit message: updated urdf

File: cad/urdf/bassie_urdf/bassie.urdf (robot description, URDF)
Before this commit: robot bassie.SLDASM, 11 links, 10 joints
Links:
- link left_ankle: geometry collision mesh filename=meshes/left_ankle.STL; visual mesh filename=meshes/left_ankle.STL
- link left_hip_pitch: geometry collision mesh filename=meshes/left_hip_pitch.STL; visual mesh filename=meshes/left_hip_pitch.STL
- link left_hip_roll: geometry collision mesh filename=meshes/left_hip_roll.STL; visual mesh filename=meshes/left_hip_roll.STL
- link left_hip_yaw: geometry collision mesh filename=meshes/left_hip_yaw.STL; visual mesh filename=meshes/left_hip_yaw.STL
- link left_knee: geometry collision mesh filename=meshes/left_knee.STL; visual mesh filename=meshes/left_knee.STL
- link pelvis: geometry collision mesh filename=meshes/pelvis.STL; visual mesh filename=meshes/pelvis.STL
- link right_ankle: geometry collision mesh filename=meshes/right_ankle.STL; visual mesh filename=meshes/right_ankle.STL
- link right_hip_pitch: geometry collision mesh filename=meshes/right_hip_pitch.STL; visual mesh filename=meshes/right_hip_pitch.STL
- link right_hip_roll: geometry collision mesh filename=meshes/right_hip_roll.STL; visual mesh filename=meshes/right_hip_roll.STL
- link right_hip_yaw: geometry collision mesh filename=meshes/right_hip_yaw.STL; visual mesh filename=meshes/right_hip_yaw.STL
- link right_knee: geometry collision mesh filename=meshes/right_knee.STL; visual mesh filename=meshes/right_knee.STL

Commit message: urdf is now correct in mujoco

File: cad/urdf/bassie_urdf/bassie.urdf (robot description, URDF)
Before this commit: robot bassie.SLDASM, 11 links, 10 joints
Links:
- removed link left_ankle
- removed link left_hip_pitch
- removed link left_hip_roll
- removed link left_hip_yaw
- removed link left_knee
- removed link right_ankle
- removed link right_hip_pitch
- removed link right_hip_roll
- removed link right_hip_yaw
- removed link right_knee
- added link left_foot, mass 0.0141163998019808; collision mesh filename=meshes/left_foot.STL; visual mesh filename=meshes/left_foot.STL
- added link left_hip_a, mass 0.0104219467105846; collision mesh filename=meshes/left_hip_a.STL; visual mesh filename=meshes/left_hip_a.STL
- added link left_hip_b, mass 0.0104219467105846; collision mesh filename=meshes/left_hip_b.STL; visual mesh filename=meshes/left_hip_b.STL
- added link left_lower_leg, mass 0.0744483650191621; collision mesh filename=meshes/left_lower_leg.STL; visual mesh filename=meshes/left_lower_leg.STL
- added link left_upper_leg, mass 0.107042315965997; collision mesh filename=meshes/left_upper_leg.STL; visual mesh filename=meshes/left_upper_leg.STL
- added link right_foot, mass 0.0141163998019807; collision mesh filename=meshes/right_foot.STL; visual mesh filename=meshes/right_foot.STL
- added link right_hip_a, mass 0.0104219467105846; collision mesh filename=meshes/right_hip_a.STL; visual mesh filename=meshes/right_hip_a.STL
- added link right_hip_b, mass 0.0104219467105846; collision mesh filename=meshes/right_hip_b.STL; visual mesh filename=meshes/right_hip_b.STL
- added link right_lower_leg, mass 0.0744483044847864; collision mesh filename=meshes/right_lower_leg.STL; visual mesh filename=meshes/right_lower_leg.STL
- added link right_upper_leg, mass 0.107018899099017; collision mesh filename=meshes/right_upper_leg.STL; visual mesh filename=meshes/right_upper_leg.STL
- link pelvis: mass 0.030372 -> 0.0303722995490468
Joints:
- joint left_ankle: child left_ankle -> left_foot; origin xyz=0 -0.18 0 rpy=-0.090229 0 0 -> xyz=0.0020029 -0.18 0 rpy=-0.074785 0 0; parent left_knee -> left_lower_leg
- joint left_hip_pitch: child left_hip_pitch -> left_hip_b; origin xyz=0 -0.014842 -0.022 rpy=-1.5708 1.5547 0 -> xyz=0 -0.020733735761258 -0.0220000000000004 rpy=-1.57079632679482 1.53550175224418 0; parent left_hip_roll -> left_hip_a
- joint left_hip_roll: child left_hip_roll -> left_hip_a; origin xyz=0.039827 0 -0.0093071 rpy=1.5708 0.21473 0 -> xyz=0.0398271658880066 0 -0.0093071036137174 rpy=1.5707963267949 0.0363921544175496 0
- joint left_hip_yaw: child left_hip_yaw -> left_upper_leg; origin xyz=0 0 -0.029158 rpy=1.4219 0 -1.5708 -> xyz=0 -0.0170842012602752 -0.0232662642387418 rpy=2.39179817705173 0 -1.5707963267949; parent left_hip_pitch -> left_hip_b
- joint left_knee: child left_knee -> left_lower_leg; origin xyz=0.021411 -0.14142 0.14142 rpy=0.16142 0 0 -> xyz=0 -0.14142 0.14142 rpy=-0.86226 0 0; parent left_hip_yaw -> left_upper_leg
- joint right_ankle: child right_ankle -> right_foot; parent right_knee -> right_lower_leg
- joint right_hip_pitch: child right_hip_pitch -> right_hip_b; origin xyz=0 -0.022001 -0.022 rpy=-1.5708 -1.4933 0 -> xyz=0 -0.0220008611326573 -0.0219999999999999 rpy=-1.57079632679503 -1.49330843492653 0; parent right_hip_roll -> right_hip_a
- joint right_hip_roll: child right_hip_roll -> right_hip_a; origin xyz=-0.039827 0 -0.0093071 rpy=1.5708 -0.0050327 0 -> xyz=-0.0398271658880066 0 -0.00930710361371741 rpy=1.5707963267949 -0.00503265783860925 0
- joint right_hip_yaw: child right_hip_yaw -> right_upper_leg; origin xyz=0 -0.021068 -0.021999 rpy=1.4762 0 1.5708 -> xyz=0 -0.0210679578739459 -0.0219991388673428 rpy=1.47617469063059 0 1.5707963267949; parent right_hip_pitch -> right_hip_b
- joint right_knee: child right_knee -> right_lower_leg; origin xyz=0 -0.14142 0.14142 rpy=0.17749 0 0 -> xyz=0 -0.14142135623731 0.141421356237308 rpy=0.177493987253612 0 0; parent right_hip_yaw -> right_upper_leg
